File: hardware-documentation/beachRover-circuit/_autosave-beachRover-circuit.sch (KiCad schematic (older format))
At the start: 3 parts

Commit message: Added few components in schematic and assigned footprints
Parts:
- removed BT1: 5v, Battery:BatteryHolder_TruPower_BH-331P_3xAA, symbol Device:Battery
- removed D1: LED, LED_THT:LED_D5.0mm, symbol Device:LED
- removed R1: 330, Resistor_THT:R_Axial_DIN0411_L9.9mm_D3.6mm_P15.24mm_Horizontal, symbol Device:R
- added A1: Arduino_Nano_v3.x, Module:Arduino_Nano_WithMountingHoles, symbol MCU_Module:Arduino_Nano_v3.x
- added J1, J2: Conn_01x02_Male, Connector_PinHeader_2.54mm:PinHeader_1x02_P2.54mm_Vertical, symbol Connector:Conn_01x02_Male
- added J3, J4: Conn_01x03, Connector_PinSocket_2.54mm:PinSocket_1x03_P2.54mm_Vertical, symbol Connector_Generic:Conn_01x03
- added J5: Barrel_Jack_Switch, Connector_BarrelJack:BarrelJack_Horizontal, symbol Connector:Barrel_Jack_Switch
- added SW1: SW_DIP_x03, Button_Switch_THT:SW_E-Switch_EG1271_DPDT, symbol Switch:SW_DIP_x03
- added U1: LM2575-5.0BT, Package_TO_SOT_THT:TO-220-5_Vertical, symbol Regulator_Switching:LM2575-5.0BT
- added U3: L293D, Package_DIP:DIP-16_W7.62mm, symbol Driver_Motor:L293D
- added U4: HC-SR04, HC-SR04:XCVR_HC-SR04, symbol HC-SR04:HC-SR04
- added U5: MMC5883MA, Package_LGA:LGA-16_3x3mm_P0.5mm, symbol Sensor_Magnetic:MMC5883MA
Connections:
- wire segments 5 -> 105
- no-connect marks 0 -> 27
